Commit message: 完成 Gazebo 阿克曼小车物理仿真调试

File: src/car_description/urdf/car.urdf.xacro (robot description, xacro)
@@ -7,3 +7,39 @@
     <!-- 引入车轮模块 -->
     <xacro:include filename="wheels.xacro"/>
+    <!-- ================= Gazebo 差速驱动插件 ================= -->
+    <gazebo>
+        <plugin name='diff_drive' filename='libgazebo_ros_diff_drive.so'>
+            <ros>
+                <namespace>/</namespace>
+                <remapping>cmd_vel:=cmd_vel</remapping>
+                <remapping>odom:=odom</remapping>
+            </ros>
+            <update_rate>50.0</update_rate>
+            <!-- 使用后轮作为驱动轮（阿克曼的前轮只能被动跟随） -->
+            <left_joint>left_rear_wheel_joint</left_joint>
+            <right_joint>right_rear_wheel_joint</right_joint>
+            <!-- 几何参数 -->
+            <wheel_separation>0.164</wheel_separation>  <!-- 轮距 -->
+            <wheel_diameter>0.049</wheel_diameter>      <!-- 车轮直径 -->
+            <!-- 速度与扭矩限制 -->
+            <max_wheel_torque>0.5</max_wheel_torque>
+            <max_wheel_acceleration>2.0</max_wheel_acceleration>    <!-- 最大轮子加速度 -->
+            <!-- 里程计与TF -->
+            <publish_odom>true</publish_odom>
+            <publish_odom_tf>true</publish_odom_tf>
+            <publish_wheel_tf>false</publish_wheel_tf>
+        </plugin>
+    </gazebo>
+     <!-- 让 Gazebo 专门发布前轮四个关节的 TF，这样 RViz 就能显示它们了 -->
+    <gazebo>
+        <plugin name="front_joint_state_publisher" filename="libgazebo_ros_joint_state_publisher.so">
+            <update_rate>50</update_rate>
+            <joint_name>left_front_steer_joint</joint_name>
+            <joint_name>right_front_steer_joint</joint_name>
+            <joint_name>left_front_wheel_joint</joint_name>
+            <joint_name>right_front_wheel_joint</joint_name>
+            <joint_name>left_rear_wheel_joint</joint_name>
+            <joint_name>right_rear_wheel_joint</joint_name>
+        </plugin>
+    </gazebo>
 </robot>

File: src/car_description/urdf/chassis.xacro (robot description, xacro)
@@ -24,3 +24,9 @@
         <xacro:box_inertia m="${chassis_mass}" x="${chassis_length}" y="${chassis_width}" z="${chassis_height}"/>
     </link>
+    <!-- Gazebo 专属标签：让底盘在仿真里是蓝色的 -->
+    <gazebo reference="base_link">
+        <material>Gazebo/Blue</material>
+        <mu1>0.2</mu1>  <!-- 底盘的摩擦系数调小，防止卡在地面上 -->
+        <mu2>0.2</mu2>
+    </gazebo>
 </robot>

File: src/car_description/urdf/wheels.xacro (robot description, xacro)
@@ -16,5 +16,5 @@
             <xacro:cylinder_inertia m="${wheel_mass}" r="${wheel_radius}" l="${wheel_width}"/>
         </link>
-        <!-- 后轮驱动关节（连续旋转） -->
+        <!-- 后轮驱动关节（连续旋转）(加入 dynamics) -->
         <joint name="${prefix}_wheel_joint" type="continuous">
             <parent link="base_link"/>
@@ -22,5 +22,5 @@
             <!-- 后轮位置：轴距的一半（负X轴），轮距的一半（Y轴镜像） -->
             <origin xyz="${-wheelbase/2} ${y_reflect * track/2} 0" rpy="1.5707 0 0"/>
-            <axis xyz="0 0 1"/>
+            <axis xyz="0 0 -1"/>
         </joint>
     </xacro:macro>
@@ -45,4 +45,6 @@
             <origin xyz="${wheelbase/2} ${y_reflect * track/2} 0" rpy="0 0 0"/>
             <axis xyz="0 0 1"/>
+            <!-- 加入阻尼，防止转向轮自发抖动 -->
+            <dynamics damping="0.5" friction="0.5"/>
             <!-- 限制最大转向角度：根据最小转弯半径0.55m和轴距0.112m计算，最大转角约0.2rad (约11.5度) -->
             <limit effort="10" lower="-0.3" upper="0.3" velocity="1.0"/>
@@ -64,8 +66,29 @@
             <child link="${prefix}_wheel_link"/>
             <origin xyz="0 0 0" rpy="1.5707 0 0"/>
-            <axis xyz="0 0 1"/>
+            <axis xyz="0 0 -1"/>
         </joint>
     </xacro:macro>
     <xacro:front_steering_wheel prefix="left_front" y_reflect="1"/>
     <xacro:front_steering_wheel prefix="right_front" y_reflect="-1"/>
+        <!-- Gazebo 专属标签：设置四个轮子的颜色和摩擦力 -->
+    <gazebo reference="left_rear_wheel_link">
+        <material>Gazebo/Black</material>
+        <mu1>1.0</mu1>  <!-- 滚动方向摩擦系数 -->
+        <mu2>1.0</mu2>  <!-- 侧滑方向摩擦系数 -->
+    </gazebo>
+    <gazebo reference="right_rear_wheel_link">
+        <material>Gazebo/Black</material>
+        <mu1>1.0</mu1>
+        <mu2>1.0</mu2>
+    </gazebo>
+    <gazebo reference="left_front_wheel_link">
+        <material>Gazebo/Black</material>
+        <mu1>1.0</mu1>
+        <mu2>1.0</mu2>
+    </gazebo>
+    <gazebo reference="right_front_wheel_link">
+        <material>Gazebo/Black</material>
+        <mu1>1.0</mu1>
+        <mu2>1.0</mu2>
+    </gazebo>
 </robot>

Commit message: docs:完成gozebo构图及整合FAST-LIO2仿真与调试流程

File: src/car_description/urdf/car.urdf.xacro (robot description, xacro)
@@ -7,6 +7,13 @@
     <!-- 引入车轮模块 -->
     <xacro:include filename="car/wheels.xacro"/>
-    <!-- 引入传感器模块 -->
-    <xacro:include filename="car/sensors.xacro"/>
+    <!-- 引入雷达模块 -->
+    <xacro:include filename="car/laser.xacro"/>
+    <!-- 引入 IMU 模块 -->
+    <xacro:include filename="car/imu.xacro"/>
+    <!-- 调用宏实例化模型 -->
+    <xacro:chassis_xacro/>
+    <xacro:wheels_xacro/>
+    <xacro:laser_xacro/>
+    <xacro:imu_xacro/>
     <!-- ================= Gazebo 差速驱动插件 ================= -->
     <gazebo>

File: src/car_description/urdf/car/chassis.xacro (robot description, xacro)
@@ -1,4 +1,4 @@
-<?xml version="1.0"?>
 <robot xmlns:xacro="http://www.ros.org/wiki/xacro">
+    <xacro:macro name="chassis_xacro">
     <!-- 根节点（地面投影） -->
     <link name="base_footprint"/>
@@ -30,3 +30,4 @@
         <mu2>0.2</mu2>
     </gazebo>
+    </xacro:macro>
 </robot>

File: src/car_description/urdf/car/wheels.xacro (robot description, xacro)
@@ -1,4 +1,4 @@
-<?xml version="1.0"?>
 <robot xmlns:xacro="http://www.ros.org/wiki/xacro">
+    <xacro:macro name="wheels_xacro" >
     <!-- ================= 1. 后轮驱动系统（后轮转向和滚动） ================= -->
     <!--prefix:部件名字前缀，y_reflect:左右镜像标志，1表示左轮，-1表示右轮-->
@@ -46,5 +46,6 @@
             <axis xyz="0 0 1"/>
             <!-- 加入阻尼，防止转向轮自发抖动 -->
-            <dynamics damping="0.5" friction="0.5"/>
+            <!-- 无法转向，暂时注释-->
+            <!--dynamics damping="0.5" friction="0.5"/-->
             <!-- 限制最大转向角度：根据最小转弯半径0.55m和轴距0.112m计算，最大转角约0.2rad (约11.5度) -->
             <limit effort="10" lower="-0.3" upper="0.3" velocity="1.0"/>
@@ -92,3 +93,4 @@
         <mu2>1.0</mu2>
     </gazebo>
+    </xacro:macro>
 </robot>

File: src/car_description/urdf/common.xacro (robot description, xacro)
@@ -1,4 +1,3 @@
-<?xml version="1.0"?>
-<robot xmlns:xacro="http://www.ros.org/wiki/xacro">
+ <robot xmlns:xacro="http://www.ros.org/wiki/xacro">
     <!-- ================= 机械尺寸参数（单位：米） ================= -->
     <!-- 底盘尺寸：230x187.6x67mm -->

Commit message: feat: 换成2D雷达，完成 2D 栅格地图建图，并集成 Nav2 导航功能

File: src/car_description/urdf/car.urdf.xacro (robot description, xacro)
@@ -11,4 +11,6 @@
     <!-- 引入 IMU 模块 -->
     <xacro:include filename="car/imu.xacro"/>
+    <!-- 引入 sonar 模块 -->
+    <xacro:include filename="car/sonar.xacro"/>
     <!-- 调用宏实例化模型 -->
     <xacro:chassis_xacro/>
@@ -16,4 +18,5 @@
     <xacro:laser_xacro/>
     <xacro:imu_xacro/>
+    <xacro:sonar_xacro/>
     <!-- ================= Gazebo 差速驱动插件 ================= -->
     <gazebo>

File: src/car_description/urdf/car/laser.xacro (robot description, xacro)
@@ -1,9 +1,9 @@
 <robot xmlns:xacro="http://www.ros.org/wiki/xacro">
     <xacro:macro name="laser_xacro">
-    <!-- ================= 1. 3D 雷达物理实体 ================= -->
+    <!-- ================= 1. 2D 雷达物理实体 ================= -->
     <link name="laser_link">
         <visual>
             <geometry>
-                <cylinder radius="0.03" length="0.04"/> <!-- 红色小圆柱体 -->
+                <cylinder radius="0.03" length="0.02"/> <!-- 红色小圆柱体 -->
             </geometry>
             <material name="red"/>
@@ -11,5 +11,5 @@
         <collision>
             <geometry>
-                <cylinder radius="0.03" length="0.04"/>
+                <cylinder radius="0.03" length="0.02"/>
             </geometry>
         </collision>
@@ -28,5 +28,5 @@
     <gazebo reference="laser_link">
         <material>Gazebo/Red</material>
-        <sensor type="ray" name="lidar3d_sensor">
+        <sensor type="ray" name="lidar2d_sensor">
             <update_rate>10</update_rate>
             <visualize>false</visualize>
@@ -34,8 +34,9 @@
                 <scan>
                     <horizontal>
-                        <samples>720</samples>
+                        <samples>360</samples>
                         <min_angle>-3.14159</min_angle>
                         <max_angle>3.14159</max_angle>
                     </horizontal>
+                    <!--
                     <vertical>
                         <samples>16</samples>
@@ -43,4 +44,5 @@
                         <max_angle>0.2618</max_angle>
                     </vertical>
+                    -->
                 </scan>
                 <range>
@@ -51,7 +53,7 @@
             <plugin name="laser_controller" filename="libgazebo_ros_ray_sensor.so">
                 <ros>
-                    <remapping>~/out:=points</remapping>
+                    <remapping>~/out:=scan</remapping>
                 </ros>
-                <output_type>sensor_msgs/PointCloud2</output_type>
+                <output_type>sensor_msgs/LaserScan</output_type>
                 <frame_name>laser_link</frame_name>
             </plugin>

File: src/car_description/urdf/car/mapping_car.xacro (robot description, xacro)
@@ -98,8 +98,8 @@
     <xacro:caster_wheel prefix="front" x_ref="0.18" />
     <xacro:caster_wheel prefix="rear"  x_ref="-0.18" />
-    <!-- ================= 3D 激光雷达 ================= -->
+    <!-- ================= 2D 激光雷达 ================= -->
     <link name="laser_link">
         <visual>
-            <geometry><cylinder radius="0.03" length="0.04"/></geometry>
+            <geometry><cylinder radius="0.03" length="0.02"/></geometry>
             <material name="red"/>
         </visual>
@@ -112,5 +112,5 @@
         <parent link="base_link"/>
         <child link="laser_link"/>
-        <origin xyz="0 0 0.09" rpy="0 0 0"/>
+        <origin xyz="0 0 0.06" rpy="0 0 0"/>
     </joint>
     <gazebo reference="laser_link">
@@ -122,8 +122,9 @@
                 <scan>
                     <horizontal>
-                        <samples>720</samples>
+                        <samples>360</samples>
                         <min_angle>-3.14159</min_angle>
                         <max_angle>3.14159</max_angle>
                     </horizontal>
+                    <!--
                     <vertical>
                         <samples>16</samples>
@@ -131,10 +132,11 @@
                         <max_angle>0.2618</max_angle>
                     </vertical>
+                    -->
                 </scan>
                 <range><min>0.1</min><max>30.0</max></range>
             </ray>
             <plugin name="laser_controller" filename="libgazebo_ros_ray_sensor.so">
-                <ros><remapping>~/out:=points</remapping></ros>
-                <output_type>sensor_msgs/PointCloud2</output_type>
+                <ros><remapping>~/out:=scan</remapping></ros>
+                <output_type>sensor_msgs/LaserScan</output_type>
                 <frame_name>laser_link</frame_name>
             </plugin>
@@ -156,5 +158,5 @@
         <sensor name="imu_sensor" type="imu">
             <always_on>true</always_on>
-            <update_rate>100</update_rate>
+            <update_rate>250</update_rate>
             <imu>
                 <angular_velocity>
@@ -173,4 +175,48 @@
                 <initial_orientation_as_reference>false</initial_orientation_as_reference>
                 <frame_name>imu_link</frame_name>
+            </plugin>
+        </sensor>
+    </gazebo>
+    <!-- ================= 3. 超声波传感器 (模拟) ================= -->
+    <link name="sonar_link">
+        <visual>
+            <geometry><sphere radius="0.01"/></geometry>
+            <material name="black"/>
+        </visual>
+        <inertial>
+            <mass value="0.05"/>
+            <inertia ixx="1e-5" ixy="0" ixz="0" iyy="1e-5" iyz="0" izz="1e-5"/>
+        </inertial>
+    </link>
+    <joint name="sonar_joint" type="fixed">
+        <parent link="base_link"/>
+        <child link="sonar_link"/>
+        <!-- 安装在车头正前方，高度与雷达相同 -->
+        <origin xyz="0.15 0 0.05" rpy="0 0 0"/>
+    </joint>
+    <gazebo reference="sonar_link">
+        <sensor type="ray" name="sonar_sensor">
+            <update_rate>20</update_rate>
+            <visualize>true</visualize>
+            <ray>
+                <scan>
+                    <horizontal>
+                        <samples>1</samples> <!-- 超声波只有一根射线 -->
+                        <min_angle>0</min_angle>
+                        <max_angle>0</max_angle>
+                    </horizontal>
+                </scan>
+                <range>
+                    <min>0.02</min> <!-- 最小 2cm -->
+                    <max>2.0</max>  <!-- 最大 2 米 -->
+                </range>
+            </ray>
+            <plugin name="sonar_controller" filename="libgazebo_ros_ray_sensor.so">
+                <ros>
+                    <!-- 话题名为 /ultrasonic -->
+                    <remapping>~/out:=ultrasonic</remapping>
+                </ros>
+                <output_type>sensor_msgs/LaserScan</output_type>
+                <frame_name>sonar_link</frame_name>
             </plugin>
         </sensor>

Commit message: RPP算法,未能正常掉头

File: src/car_description/urdf/car.urdf.xacro (robot description, xacro)
@@ -19,7 +19,7 @@
     <xacro:imu_xacro/>
     <xacro:sonar_xacro/>
-    <!-- ================= Gazebo 差速驱动插件 ================= -->
+        <!-- ================= 1. 阿克曼专属驱动插件 ================= -->
     <gazebo>
-        <plugin name='diff_drive' filename='libgazebo_ros_diff_drive.so'>
+        <plugin name="ackermann_drive" filename="libgazebo_ros_ackermann_drive.so">
             <ros>
                 <namespace>/</namespace>
@@ -27,24 +27,29 @@
                 <remapping>odom:=odom</remapping>
             </ros>
-            <update_rate>50.0</update_rate>
-            <!-- 使用后轮作为驱动轮（阿克曼的前轮只能被动跟随） -->
-            <left_joint>left_rear_wheel_joint</left_joint>
-            <right_joint>right_rear_wheel_joint</right_joint>
-            <!-- 几何参数 -->
-            <wheel_separation>0.164</wheel_separation>  <!-- 轮距 -->
-            <wheel_diameter>0.049</wheel_diameter>      <!-- 车轮直径 -->
-            <!-- 速度与扭矩限制 -->
-            <max_wheel_torque>0.5</max_wheel_torque>
-            <max_wheel_acceleration>2.0</max_wheel_acceleration>    <!-- 最大轮子加速度 -->
-            <!-- 里程计与TF -->
+            <update_rate>30.0</update_rate>
+            <!-- 🔥 注意这里的参数名：必须写全，且与你 wheels.xacro 里的关节名绝对一致！ -->
+            <left_steering_joint>left_front_steer_joint</left_steering_joint>
+            <right_steering_joint>right_front_steer_joint</right_steering_joint>
+            <left_rear_wheel_joint>left_rear_wheel_joint</left_rear_wheel_joint>
+            <right_rear_wheel_joint>right_rear_wheel_joint</right_rear_wheel_joint>
+            <!-- 几何尺寸 -->
+            <wheelbase>0.112</wheelbase>
+            <wheel_separation>0.164</wheel_separation>
+            <wheel_radius>0.0245</wheel_radius>
+            <!-- 核心：内置 PID 控制前轮，专治各种抽搐、抖动 -->
+            <max_speed>1.5</max_speed>
+            <max_steer>0.5</max_steer>
+            <kp>100.0</kp>
+            <kd>10.0</kd>
             <publish_odom>true</publish_odom>
             <publish_odom_tf>true</publish_odom_tf>
-            <publish_wheel_tf>false</publish_wheel_tf>
         </plugin>
     </gazebo>
-     <!-- 让 Gazebo 专门发布前轮四个关节的 TF，这样 RViz 就能显示它们了 -->
+    <!-- ================= 2. 关节状态发布插件 (必须加回来！) ================= -->
+    <!-- 它的唯一任务是读取物理引擎的状态，发给 robot_state_publisher -->
     <gazebo>
-        <plugin name="front_joint_state_publisher" filename="libgazebo_ros_joint_state_publisher.so">
+        <plugin name="joint_state_publisher" filename="libgazebo_ros_joint_state_publisher.so">
             <update_rate>50</update_rate>
+            <!-- 发布所有轮子和转向关节的状态 -->
             <joint_name>left_front_steer_joint</joint_name>
             <joint_name>right_front_steer_joint</joint_name>

File: src/car_description/urdf/car/wheels.xacro (robot description, xacro)
@@ -22,5 +22,5 @@
             <!-- 后轮位置：轴距的一半（负X轴），轮距的一半（Y轴镜像） -->
             <origin xyz="${-wheelbase/2} ${y_reflect * track/2} 0" rpy="1.5707 0 0"/>
-            <axis xyz="0 0 -1"/>
+            <axis xyz="0 0 ${-y_reflect}"/>
         </joint>
     </xacro:macro>
@@ -45,9 +45,8 @@
             <origin xyz="${wheelbase/2} ${y_reflect * track/2} 0" rpy="0 0 0"/>
             <axis xyz="0 0 1"/>
-            <!-- 加入阻尼，防止转向轮自发抖动 -->
-            <!-- 无法转向，暂时注释-->
-            <!--dynamics damping="0.5" friction="0.5"/-->
+            <!-- 加入阻尼和摩擦，防止转向轮自发抖动 -->
+            <dynamics damping="2.0" friction="0.5"/>
             <!-- 限制最大转向角度：根据最小转弯半径0.55m和轴距0.112m计算，最大转角约0.2rad (约11.5度) -->
-            <limit effort="10" lower="-0.3" upper="0.3" velocity="1.0"/>
+            <limit effort="10" lower="-0.5" upper="0.5" velocity="1.0"/>
         </joint>
         <!-- 前轮轮子 -->
@@ -67,5 +66,5 @@
             <child link="${prefix}_wheel_link"/>
             <origin xyz="0 0 0" rpy="1.5707 0 0"/>
-            <axis xyz="0 0 -1"/>
+            <axis xyz="0 0 ${-y_reflect}"/>
         </joint>
     </xacro:macro>

Commit message: refactor(car): 新增 car_bringup 包统一管理启动文件与导航参数
- 将 launch 文件、nav2 参数和地图从 car_description/car_navigation 迁移至 car_bringup
- URDF 中移除内联的阿克曼驱动插件，拆分至 control.xacro 并引入 ros2_control
- 修正车轮关节轴向定义，统一为 -z 并补充 effort/velocity 限制
- 调整转向关节限位为 ±0.235 rad，更新轮子摩擦参数与 RViz 固定坐标系为 odom

File: src/car_description/urdf/car.urdf.xacro (robot description, xacro)
@@ -13,4 +13,6 @@
     <!-- 引入 sonar 模块 -->
     <xacro:include filename="car/sonar.xacro"/>
+    <!-- 引入控制模块 -->
+    <xacro:include filename="car/control.xacro"/>
     <!-- 调用宏实例化模型 -->
     <xacro:chassis_xacro/>
@@ -19,44 +21,3 @@
     <xacro:imu_xacro/>
     <xacro:sonar_xacro/>
-        <!-- ================= 1. 阿克曼专属驱动插件 ================= -->
-    <gazebo>
-        <plugin name="ackermann_drive" filename="libgazebo_ros_ackermann_drive.so">
-            <ros>
-                <namespace>/</namespace>
-                <remapping>cmd_vel:=cmd_vel</remapping>
-                <remapping>odom:=odom</remapping>
-            </ros>
-            <update_rate>30.0</update_rate>
-            <!-- 🔥 注意这里的参数名：必须写全，且与你 wheels.xacro 里的关节名绝对一致！ -->
-            <left_steering_joint>left_front_steer_joint</left_steering_joint>
-            <right_steering_joint>right_front_steer_joint</right_steering_joint>
-            <left_rear_wheel_joint>left_rear_wheel_joint</left_rear_wheel_joint>
-            <right_rear_wheel_joint>right_rear_wheel_joint</right_rear_wheel_joint>
-            <!-- 几何尺寸 -->
-            <wheelbase>0.112</wheelbase>
-            <wheel_separation>0.164</wheel_separation>
-            <wheel_radius>0.0245</wheel_radius>
-            <!-- 核心：内置 PID 控制前轮，专治各种抽搐、抖动 -->
-            <max_speed>1.5</max_speed>
-            <max_steer>0.5</max_steer>
-            <kp>100.0</kp>
-            <kd>10.0</kd>
-            <publish_odom>true</publish_odom>
-            <publish_odom_tf>true</publish_odom_tf>
-        </plugin>
-    </gazebo>
-    <!-- ================= 2. 关节状态发布插件 (必须加回来！) ================= -->
-    <!-- 它的唯一任务是读取物理引擎的状态，发给 robot_state_publisher -->
-    <gazebo>
-        <plugin name="joint_state_publisher" filename="libgazebo_ros_joint_state_publisher.so">
-            <update_rate>50</update_rate>
-            <!-- 发布所有轮子和转向关节的状态 -->
-            <joint_name>left_front_steer_joint</joint_name>
-            <joint_name>right_front_steer_joint</joint_name>
-            <joint_name>left_front_wheel_joint</joint_name>
-            <joint_name>right_front_wheel_joint</joint_name>
-            <joint_name>left_rear_wheel_joint</joint_name>
-            <joint_name>right_rear_wheel_joint</joint_name>
-        </plugin>
-    </gazebo>
 </robot>

File: src/car_description/urdf/car/wheels.xacro (robot description, xacro)
@@ -21,6 +21,9 @@
             <child link="${prefix}_wheel_link"/>
             <!-- 后轮位置：轴距的一半（负X轴），轮距的一半（Y轴镜像） -->
+            <!-- rpy=+90° 后，关节局部 +z 指向世界 -y；取 -z 才能让
+                 “正速度 = 车向前 (+x)” 与控制器/里程计符号一致 -->
             <origin xyz="${-wheelbase/2} ${y_reflect * track/2} 0" rpy="1.5707 0 0"/>
-            <axis xyz="0 0 ${-y_reflect}"/>
+            <axis xyz="0 0 -1"/>
+            <limit effort="10.0" velocity="45.0"/>
         </joint>
     </xacro:macro>
@@ -47,6 +50,6 @@
             <!-- 加入阻尼和摩擦，防止转向轮自发抖动 -->
             <dynamics damping="2.0" friction="0.5"/>
-            <!-- 限制最大转向角度：根据最小转弯半径0.55m和轴距0.112m计算，最大转角约0.2rad (约11.5度) -->
-            <limit effort="10" lower="-0.5" upper="0.5" velocity="1.0"/>
+            <!-- 限制最大转向角度-->
+            <limit effort="10" lower="-0.235" upper="0.235" velocity="2.0"/>
         </joint>
         <!-- 前轮轮子 -->
@@ -66,5 +69,6 @@
             <child link="${prefix}_wheel_link"/>
             <origin xyz="0 0 0" rpy="1.5707 0 0"/>
-            <axis xyz="0 0 ${-y_reflect}"/>
+            <axis xyz="0 0 -1"/>
+            <limit effort="10.0" velocity="45.0"/>
         </joint>
     </xacro:macro>
@@ -82,4 +86,6 @@
         <mu2>1.0</mu2>
     </gazebo>
+    <!-- 阿克曼车的四个轮子都需要足够的侧向抓地力（mu2），
+         前轮 mu2=0.1 会让车头侧滑、无法按转角转弯 -->
     <gazebo reference="left_front_wheel_link">
         <material>Gazebo/Black</material>

File: src/car_description/urdf/common.xacro (robot description, xacro)
@@ -20,4 +20,5 @@
     <material name="black"><color rgba="0 0 0 1"/></material>
     <material name="red"><color rgba="1 0 0 1"/></material>
+    <material name="green"><color rgba="0 1 0 1"/></material>
     <!-- ================= 惯性矩阵宏 ================= -->
     <xacro:macro name="box_inertia" params="m x y z">
