Commit message: feat(control): 新增 r5_steering_controller 及实车参数修正与验收脚本

File: src/car_description/urdf/car/control.xacro (robot description, xacro)
@@ -45,12 +45,12 @@
             <parameters>$(find car_bringup)/config/controllers.yaml</parameters>
             <ros>
-                <!-- 重映射一些官方控制器的话题 -->
-                <remapping>/ackermann_steering_controller/tf_odometry:=/tf</remapping>
-                <remapping>/ackermann_steering_controller/odometry:=/odom</remapping>
+                <!-- 重映射一些官方控制器的话题（控制器改名为 r5_steering_controller 后同步改） -->
+                <remapping>/r5_steering_controller/tf_odometry:=/tf</remapping>
+                <remapping>/r5_steering_controller/odometry:=/odom</remapping>
                 <!-- controllers.yaml 中 use_stamped_vel 为 false 时控制器订阅
                      ~/reference_unstamped；这里把它映射成标准的 /cmd_vel -->
                 <!-- 注意：URDF 注释里不要出现 ASCII 的“冒号+空格”，
                      gazebo_ros2_control 会把 robot_description 当作参数覆盖规则解析 -->
-                <remapping>/ackermann_steering_controller/reference_unstamped:=/cmd_vel</remapping>
+                <remapping>/r5_steering_controller/reference_unstamped:=/cmd_vel</remapping>
             </ros>
         </plugin>

File: src/car_description/urdf/car/wheels.xacro (robot description, xacro)
@@ -50,6 +50,8 @@
             <!-- 加入阻尼和摩擦，防止转向轮自发抖动 -->
             <dynamics damping="2.0" friction="0.5"/>
-            <!-- 限制最大转向角度-->
-            <limit effort="10" lower="-0.235" upper="0.235" velocity="2.0"/>
+            <!-- 实车依据（手册参数表）：最小转弯半径 0.55m → 内侧前轮
+                 atan(0.112/(0.55-0.082)) ≈ 0.235 rad（外侧 0.176 rad）；
+                 舵机 S620F-180 响应 0.11s/60° ≈ 9.5 rad/s -->
+            <limit effort="10" lower="-0.235" upper="0.235" velocity="9.5"/>
         </joint>
         <!-- 前轮轮子 -->

File: src/car_description/urdf/common.xacro (robot description, xacro)
@@ -8,12 +8,14 @@
     <xacro:property name="wheelbase" value="0.112"/>
     <xacro:property name="track" value="0.164"/>
-    <!-- 车轮尺寸：直径49mm，宽度45mm -->
-    <xacro:property name="wheel_radius" value="0.0245"/>
+    <!-- 车轮尺寸：手册参数表为 65mm 橡胶轮胎（与“330rpm×1.2m/s”反推一致）；
+         图纸上的 49 标注疑为轮毂直径。TODO：拿实物量外径确认，
+         若实测不是 65 只需改这一个数（轮径直接乘进里程计和最大车速）。 -->
+    <xacro:property name="wheel_radius" value="0.0325"/>
     <xacro:property name="wheel_width" value="0.045"/>
     <!-- ================= 质量参数（总重0.9kg） ================= -->
     <xacro:property name="chassis_mass" value="0.8"/> <!-- 底盘重0.8kg -->
     <xacro:property name="wheel_mass" value="0.025"/> <!-- 每个轮子0.025kg，4个合计0.1kg -->
-    <!-- 底盘离地高度（让车轮刚好接触地面） -->
-    <xacro:property name="chassis_z_offset" value="0.0245"/>
+    <!-- 底盘离地高度（让车轮刚好接触地面） = 轮半径 -->
+    <xacro:property name="chassis_z_offset" value="${wheel_radius}"/>
     <!-- ================= 材质定义 ================= -->
     <material name="blue"><color rgba="0 0 1 1"/></material>
